File: pcb/bully.kicad_sch (KiCad schematic)
At the start: 29 parts, among them J1 SM04B-SRSS-TB(LF)(SN), J2 Conn_01x04, U1 W25Q128JVS, U3 RP2040, U4 XC6206PxxxMR-Regulator_Linear, Y1 12MHz

Commit message: updated bom
Parts:
- C1, C10, C11, C12, C13, C14, C15, C5, C6, C9: LCSC C1525 -> (none)
- C16, C17, C4, C8: LCSC C52923 -> (none)
- C2, C3: LCSC C1555 -> (none)
- C7: LCSC C15525 -> (none)
- R1, R7: LCSC C11702 -> (none)
- R5, R6: LCSC C25190 -> (none)
- SW_BOOT1, SW_RST1: value SW_Push -> SKQGABE010
Changed lines of the file:
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@@
       (effects (font (size 1.27 1.27)) hide)
     )
-    (property "LCSC" "C1525" (at 147.32 53.34 0)
+    (property "LCSC" "" (at 147.32 53.34 0)
       (effects (font (size 1.27 1.27)) hide)
     )
@@
       (effects (font (size 1.27 1.27)))
     )
-    (property "Value" "SW_Push" (at 245.745 55.88 0)
+    (property "Value" "SKQGABE010" (at 245.745 55.88 0)
       (effects (font (size 1.27 1.27)))
     )
@@
       (effects (font (size 1.27 1.27)) hide)
     )
-    (property "LCSC" "C15525" (at 113.03 53.34 0)
+    (property "LCSC" "" (at 113.03 53.34 0)
       (effects (font (size 1.27 1.27)) hide)
     )
@@
       (effects (font (size 1.27 1.27)) hide)
     )
-    (property "LCSC" "C1525" (at 173.99 53.34 0)
+    (property "LCSC" "" (at 173.99 53.34 0)
       (effects (font (size 1.27 1.27)) hide)
     )
@@
       (effects (font (size 1.27 1.27)))
     )
-    (property "Value" "SW_Push" (at 245.745 32.385 0)
+    (property "Value" "SKQGABE010" (at 245.745 32.385 0)
       (effects (font (size 1.27 1.27)))
     )
@@
       (effects (font (size 1.27 1.27)) hide)
     )
-    (property "LCSC" "C52923" (at 113.03 30.48 0)
+    (property "LCSC" "" (at 113.03 30.48 0)
       (effects (font (size 1.27 1.27)) hide)
     )
@@
       (effects (font (size 1.27 1.27)) hide)
     )
-    (property "LCSC" "C1525" (at 143.51 80.645 0)
+    (property "LCSC" "" (at 143.51 80.645 0)
       (effects (font (size 1.27 1.27)) hide)
     )
@@
       (effects (font (size 1.27 1.27)) hide)
     )
-    (property "LCSC" "C1555" (at 122.555 159.385 0)
+    (property "LCSC" "" (at 122.555 159.385 0)
       (effects (font (size 1.27 1.27)) hide)
     )
@@
       (effects (font (size 1.27 1.27)) hide)
     )
-    (property "LCSC" "C52923" (at 149.098 132.842 0)
+    (property "LCSC" "" (at 149.098 132.842 0)
       (effects (font (size 1.27 1.27)) hide)
     )
@@
       (effects (font (size 1.27 1.27)) hide)
     )
-    (property "LCSC" "C1525" (at 165.1 53.34 0)
+    (property "LCSC" "" (at 165.1 53.34 0)
       (effects (font (size 1.27 1.27)) hide)
     )
@@
       (effects (font (size 1.27 1.27)) hide)
     )
-    (property "LCSC" "C52923" (at 117.602 132.842 0)
+    (property "LCSC" "" (at 117.602 132.842 0)
       (effects (font (size 1.27 1.27)) hide)
     )
@@
       (effects (font (size 1.27 1.27)) hide)
     )
-    (property "LCSC" "C1555" (at 122.555 154.305 0)
+    (property "LCSC" "" (at 122.555 154.305 0)
       (effects (font (size 1.27 1.27)) hide)
     )
@@
       (effects (font (size 1.27 1.27)) hide)
     )
-    (property "LCSC" "C1525" (at 138.43 53.34 0)
+    (property "LCSC" "" (at 138.43 53.34 0)
       (effects (font (size 1.27 1.27)) hide)
     )
@@
       (effects (font (size 1.27 1.27)) hide)
     )
-    (property "LCSC" "C1525" (at 129.54 53.34 0)
+    (property "LCSC" "" (at 129.54 53.34 0)
       (effects (font (size 1.27 1.27)) hide)
     )
@@
       (effects (font (size 1.27 1.27)) hide)
     )
-    (property "LCSC" "C1525" (at 156.21 53.34 0)
+    (property "LCSC" "" (at 156.21 53.34 0)
       (effects (font (size 1.27 1.27)) hide)
     )
@@
       (effects (font (size 1.27 1.27)) hide)
     )
-    (property "LCSC" "C11702" (at 121.285 93.345 0)
+    (property "LCSC" "" (at 121.285 93.345 0)
       (effects (font (size 1.27 1.27)) hide)
     )
@@
       (effects (font (size 1.27 1.27)) hide)
     )
-    (property "LCSC" "C25190" (at 33.02 66.675 0)
+    (property "LCSC" "" (at 33.02 66.675 0)
       (effects (font (size 1.27 1.27)) hide)
     )
@@
       (effects (font (size 1.27 1.27)) hide)
     )
-    (property "LCSC" "C25190" (at 33.02 69.215 0)
+    (property "LCSC" "" (at 33.02 69.215 0)
       (effects (font (size 1.27 1.27)) hide)
     )
@@
       (effects (font (size 1.27 1.27)) hide)
     )
-    (property "LCSC" "C1525" (at 119.38 30.48 0)
+    (property "LCSC" "" (at 119.38 30.48 0)
       (effects (font (size 1.27 1.27)) hide)
     )
@@
       (effects (font (size 1.27 1.27)) hide)
     )
-    (property "LCSC" "C1525" (at 120.65 53.34 0)
+    (property "LCSC" "" (at 120.65 53.34 0)
       (effects (font (size 1.27 1.27)) hide)
     )
@@
       (effects (font (size 1.27 1.27)) hide)
     )
-    (property "LCSC" "C1525" (at 128.27 30.48 0)
+    (property "LCSC" "" (at 128.27 30.48 0)
       (effects (font (size 1.27 1.27)) hide)
     )
@@
       (effects (font (size 1.27 1.27)) hide)
     )
-    (property "LCSC" "C52923" (at 125.222 132.842 0)
+    (property "LCSC" "" (at 125.222 132.842 0)
       (effects (font (size 1.27 1.27)) hide)
     )
@@
       (effects (font (size 1.27 1.27)) hide)
     )
-    (property "LCSC" "C11702" (at 144.145 159.385 0)
-      (effects (font (size 1.27 1.27)) hide)
-    )
+    (property "LCSC" "" (at 144.145 159.385 0)
+      (effects (font (size 1.27 1.27)) hide)
+    )
