File: pcb/bully.kicad_pcb (KiCad board)
At the start: 2 copper layers, 257.2 x 89.2 mm, 137 parts, among them J1 SM04B-SRSS-TB(LF)(SN), J2 Conn_01x04, SW1 SW_Push, SW10 SW_Push, SW11 SW_Push, SW12 SW_Push, SW13 SW_Push, SW14 SW_Push, SW15 SW_Push, SW16 SW_Push, SW17 SW_Push, SW18 SW_Push, SW19 SW_Push, SW2 SW_Push, SW20 SW_Push, SW21 SW_Push, SW22 SW_Push, SW23 SW_Push, SW24 SW_Push, SW25 SW_Push, SW26 SW_Push, SW27 SW_Push, SW28 SW_Push, SW29 SW_Push, SW3 SW_Push, SW30 SW_Push, SW31 SW_Push, SW32 SW_Push, SW33 SW_Push, SW34 SW_Push, SW35 SW_Push, SW36 SW_Push, SW37 SW_Push, SW38 SW_Push, SW39 SW_Push, SW4 SW_Push, SW40 SW_Push, SW41 SW_Push, SW42 SW_Push, SW43 SW_Push, SW44 SW_Push, SW45 SW_Push, SW46 SW_Push, SW47 SW_Push, SW48 SW_Push, SW49 SW_Push, SW5 SW_Push, SW50 SW_Push, SW51 SW_Push, SW52 SW_Push, SW53 SW_Push, SW54 SW_Push, SW55 SW_Push, SW56 SW_Push, SW6 SW_Push, SW7 SW_Push, SW8 SW_Push, SW9 SW_Push, U1 W25Q128JVS, U3 RP2040, U4 XC6206PxxxMR-Regulator_Linear, Y1 12MHz

Commit message: Added 150/225 bottom row for hhkb support
Fixed positions of many bottom row alternate layouts. No BOM changes, just moved one diode and a few conflicting traces.
Gerbers have been updated
Parts:
- added SW57: SW_Push, MX_Solderable:MX-Solderable-1.5U, F.Cu at (57.5, 120.3)
- added SW58: SW_Push, MX_Solderable:MX-Solderable-2.25U-ReversedStabilizers, F.Cu at (93.2, 120.3)
- added SW59: SW_Push, MX_Solderable:MX-Solderable-2.25U-ReversedStabilizers, F.Cu at (202.7, 120.3)
- added SW60: SW_Push, MX_Solderable:MX-Solderable-1.5U, F.Cu at (238.4, 120.3)
- SW_BOOT1, SW_RST1: value SW_Push -> SKQGABE010
- moved SW55 2.38 mm to (157.5, 120.3)
- moved D49 2.00 mm to (219.0, 111.5)
- moved SW54 0.18 mm to (138.5, 120.3)
Connections:
- SW53 pad 1: COL4 -> Net-(D43-A)
- SW53 pad 2: Net-(D43-A) -> COL4
- SW56 pad 1: COL10 -> Net-(D49-A)
- SW56 pad 2: Net-(D49-A) -> COL10
Routing:
- net Net-(D49-A): track 15.0 -> 28.8 mm
- net COL4: track 157.4 -> 168.4 mm
- net Net-(D42-A): track 4.62 -> 14.1 mm
- net COL3: track 165.5 -> 175.0 mm
- net COL11: track 112.9 -> 122.4 mm
- net Net-(D46-A): track 20.8 -> 27.8 mm
- net COL7: track 89.1 -> 95.6 mm
- net Net-(D50-A): track 5.46 -> 11.2 mm
- net COL10: track 103.0 -> 101.5 mm
